Commit message: created jazzy migrat branch

File: src/simulations/robot_gazebo/urdf/imu.gazebo.xacro (robot description, xacro)
@@ -5,5 +5,5 @@
             <always_on>1</always_on>
             <update_rate>50</update_rate>
-            <ignition_frame_id>imu_link</ignition_frame_id>
+            <gz_frame_id>imu_link</gz_frame_id>
             <visualize>true</visualize>
             <topic>imu</topic>

File: src/simulations/robot_gazebo/urdf/lidar.gazebo.xacro (robot description, xacro)
@@ -6,5 +6,5 @@
             <topic>scan</topic>
             <update_rate>10</update_rate>
-            <ignition_frame_id>lidar_link</ignition_frame_id>
+            <gz_frame_id>lidar_link</gz_frame_id>
             <ray>
                 <scan>
@@ -27,5 +27,5 @@
                 </noise>
             </ray>
-            <alwaysOn>1</alwaysOn>
+            <always_on>1</always_on>
             <visualize>true</visualize>
         </sensor>

File: src/simulations/robot_gazebo/urdf/rospider.gazebo.xacro (robot description, xacro)
@@ -1,3 +1,19 @@
 <?xml version="1.0" encoding="utf-8"?>
+<!--
+  MIGRATED Humble to Jazzy.
+  REMOVED: <param name="mimic"> and <param name="multiplier"> from every joint.
+  Jazzy's ros2_control deleted these; mimic is now read ONLY from the <mimic>
+  tag in the URDF joint definition (rospider_description/urdf/gripper.urdf.xacro).
+  !! ACTION REQUIRED - the two sources DISAGREED, so behavior will change !!
+      joint        | this file said  | gripper.urdf.xacro says
+      l_joint      | r_joint x (-1)  | r_joint x (-1)   agree
+      l_in_joint   | l_joint x (+1)  | r_joint x (-1)   agree, via l_joint
+      l_out_joint  | l_joint x (+1)  | r_joint x (-1)   agree, via l_joint
+      r_in_joint   | r_joint x (+1)  | r_joint x (-1)   CONFLICT
+      r_out_joint  | r_joint x (-1)  | r_joint x (+1)   CONFLICT
+  On Humble this file won. On Jazzy the URDF wins, so r_in_joint and
+  r_out_joint will move in the OPPOSITE direction from before. Decide which
+  is correct and edit the <mimic> tags in gripper.urdf.xacro accordingly.
+-->
 <robot name="arm" xmlns:xacro="http://ros.org/wiki/xacro">
   <ros2_control name="GazeboSystem" type="system">
@@ -57,29 +73,21 @@
       <state_interface name="effort"/>
     </joint>
-    <joint name="l_joint"> <param name="mimic">r_joint</param>
-      <param name="multiplier">-1</param>
-      <state_interface name="position"/>
-      <state_interface name="velocity"/>
-      <state_interface name="effort"/>
-    </joint>
-    <joint name="l_in_joint"> <param name="mimic">l_joint</param>
-      <param name="multiplier">1</param>
-      <state_interface name="position"/>
-      <state_interface name="velocity"/>
-      <state_interface name="effort"/>
-    </joint>
-    <joint name="l_out_joint"> <param name="mimic">l_joint</param>
-      <param name="multiplier">1</param> <state_interface name="position"/>
-      <state_interface name="velocity"/>
-      <state_interface name="effort"/>
-    </joint>
-    <joint name="r_in_joint"> <param name="mimic">r_joint</param>
-      <param name="multiplier">1</param>
-      <state_interface name="position"/>
-      <state_interface name="velocity"/>
-      <state_interface name="effort"/>
-    </joint>
-    <joint name="r_out_joint"> <param name="mimic">r_joint</param>
-      <param name="multiplier">-1</param> <state_interface name="position"/>
+    <joint name="l_joint"><state_interface name="position"/>
+      <state_interface name="velocity"/>
+      <state_interface name="effort"/>
+    </joint>
+    <joint name="l_in_joint"><state_interface name="position"/>
+      <state_interface name="velocity"/>
+      <state_interface name="effort"/>
+    </joint>
+    <joint name="l_out_joint"><state_interface name="position"/>
+      <state_interface name="velocity"/>
+      <state_interface name="effort"/>
+    </joint>
+    <joint name="r_in_joint"><state_interface name="position"/>
+      <state_interface name="velocity"/>
+      <state_interface name="effort"/>
+    </joint>
+    <joint name="r_out_joint"><state_interface name="position"/>
       <state_interface name="velocity"/>
       <state_interface name="effort"/>
